Commit message: [BSAP]TASK: project to local path.

File: src/planning_core/urdf/tp_model/tp_car.xacro (robot description, xacro)
@@ -1,4 +1,5 @@
 <!-- Chassis -->
 <robot xmlns:xacro="http://www.ros.org/wiki/xacro" name="tp_car">
+    <xacro:property name="use_dynamic_tps_config" value="true"/>
     <!-- Color-->
     <material name="blue">
@@ -21,5 +22,5 @@
         </link>
         <!-- projection point to the map -->
-        <joint name="{footprint${id}_to_map" type="fixed">
+        <joint name="footprint${id}_to_map" type="fixed">
             <parent link="map"/>
             <child link="base_footprint_tp${id}"/>
@@ -33,6 +34,15 @@
     </xacro:macro>
     <!-- function call -->
-    <xacro:create_tp_car id="1" car_length="3.0" car_width="1.6" car_height="1.2" color="blue"/>
-    <xacro:create_tp_car id="2" car_length="3.0" car_width="1.6" car_height="1.2" color="blue"/>
-    <xacro:create_tp_car id="3" car_length="3.0" car_width="1.6" car_height="1.2" color="blue"/>
+    <!-- static tps config -->
+    <xacro:if value="${not use_dynamic_tps_config}">
+      <xacro:create_tp_car id="1" car_length="3.0" car_width="1.6" car_height="1.2" color="blue"/>
+      <xacro:create_tp_car id="2" car_length="3.0" car_width="1.6" car_height="1.2" color="blue"/>
+      <xacro:create_tp_car id="3" car_length="3.0" car_width="1.6" car_height="1.2" color="blue"/>
+    </xacro:if>
+    <!-- dynamic tps config -->
+    <xacro:if value="${use_dynamic_tps_config}">
+      <xacro:create_tp_car id="1" car_length="8.0" car_width="2.6" car_height="1.2" color="blue"/>
+      <xacro:create_tp_car id="2" car_length="6.0" car_width="2.0" car_height="1.2" color="blue"/>
+      <xacro:create_tp_car id="3" car_length="3.0" car_width="7.6" car_height="1.2" color="blue"/>
+    </xacro:if>
 </robot>

Commit message: Add planning configuration files for in-lane traffic planning scenarios
- Created `planning_inlane_tps_config.yaml` to define vehicle parameters, map characteristics, path configurations, decision margins, and movement commands for in-lane traffic planning.
- Added `scenario_config.yaml` to specify the type of scenario and the number of traffic participants for testing different planning strategies.

File: src/planning_core/urdf/tp_model/tp_car.xacro (robot description, xacro)
@@ -1,5 +1,7 @@
 <!-- Chassis -->
 <robot xmlns:xacro="http://www.ros.org/wiki/xacro" name="tp_car">
-    <xacro:property name="use_dynamic_tps_config" value="true"/>
+    <xacro:arg name="tp_num" default="3"/>
+    <xacro:property name="tp_count" value="$(arg tp_num)"/>
+    <xacro:property name="use_dynamic_tps_config" value="false"/>
     <!-- Color-->
     <material name="blue">
@@ -33,16 +35,28 @@
         </joint>
     </xacro:macro>
-    <!-- function call -->
+    <!-- function call, controlled by tp_num arg -->
     <!-- static tps config -->
     <xacro:if value="${not use_dynamic_tps_config}">
-      <xacro:create_tp_car id="1" car_length="3.0" car_width="1.6" car_height="1.2" color="blue"/>
-      <xacro:create_tp_car id="2" car_length="3.0" car_width="1.6" car_height="1.2" color="blue"/>
-      <xacro:create_tp_car id="3" car_length="3.0" car_width="1.6" car_height="1.2" color="blue"/>
+      <xacro:if value="${int(tp_count) >= 1}">
+        <xacro:create_tp_car id="1" car_length="3.0" car_width="1.6" car_height="1.2" color="blue"/>
+      </xacro:if>
+      <xacro:if value="${int(tp_count) >= 2}">
+        <xacro:create_tp_car id="2" car_length="3.0" car_width="1.6" car_height="1.2" color="blue"/>
+      </xacro:if>
+      <xacro:if value="${int(tp_count) >= 3}">
+        <xacro:create_tp_car id="3" car_length="3.0" car_width="1.6" car_height="1.2" color="blue"/>
+      </xacro:if>
     </xacro:if>
     <!-- dynamic tps config -->
     <xacro:if value="${use_dynamic_tps_config}">
-      <xacro:create_tp_car id="1" car_length="8.0" car_width="2.6" car_height="1.2" color="blue"/>
-      <xacro:create_tp_car id="2" car_length="6.0" car_width="2.0" car_height="1.2" color="blue"/>
-      <xacro:create_tp_car id="3" car_length="3.0" car_width="7.6" car_height="1.2" color="blue"/>
+      <xacro:if value="${int(tp_count) >= 1}">
+        <xacro:create_tp_car id="1" car_length="8.0" car_width="2.6" car_height="1.2" color="blue"/>
+      </xacro:if>
+      <xacro:if value="${int(tp_count) >= 2}">
+        <xacro:create_tp_car id="2" car_length="6.0" car_width="2.0" car_height="1.2" color="blue"/>
+      </xacro:if>
+      <xacro:if value="${int(tp_count) >= 3}">
+        <xacro:create_tp_car id="3" car_length="3.0" car_width="7.6" car_height="1.2" color="blue"/>
+      </xacro:if>
     </xacro:if>
 </robot>
